Commit message: Add Effort/ Velocity/ Position Controllers

File: urdf/cartpole_v0.urdf (robot description, URDF)
Before this commit: robot cartpole_v0, 4 links, 3 joints
Links:
- link bar_link: mass 1 -> 5
Joints:
- joint joint_1: limit lower=-1.57 upper=1.57 effort=2000000 velocity=10000 -> lower=-1.57 upper=1.57 effort=200 velocity=100
- joint joint_2: limit lower=-2.0 upper=2.0 effort=2000000 velocity=100000 -> lower=-2.0 upper=2.0 effort=200 velocity=100
